File: Dual_Bios_Switch_Board/Dual_Bios_Switch_Board.kicad_pcb (KiCad board)
At the start: 2 copper layers, 22.4 x 23 mm, 6 parts, among them J1 Conn_02x04_Counter_Clockwise, SW1 SW_DPDT_x2, U1 SOIC-8, U2 SOIC-8

Commit message: adjust some details issues
Parts:
- moved U1 1.12 mm to (204.0, 145.5)
- moved U2 1.12 mm to (204.0, 133.5)
Routing:
- net DI: track 24.0 -> 18.9 mm
- net DO: track 26.4 -> 25.0 mm
- net WP: track 28.2 -> 27.0 mm
- net CS1: track 13.4 -> 14.4 mm
- net CS2: track 14.6 -> 15.4 mm
Other:
- board size 22.4 x 23 mm -> 23.4 x 21.5 mm
